File: src/PCB_Design.kicad_sch (KiCad schematic)
At the start: 9 parts, among them U1 ADS1299xPAG

Commit message: Schematic
Parts:
- added C10, C15, C16, C8, C9: 1μF, Capacitor_SMD:C_0402_1005Metric, symbol Device:C
- added C11, C13, C5, C6: 0.1μF, Capacitor_SMD:C_0402_1005Metric, symbol Device:C
- added C12: 1nF, Capacitor_SMD:C_0402_1005Metric, symbol Device:C
- added C14: 10μF, Capacitor_SMD:C_0402_1005Metric, symbol Device:C
- added C7: 100μF, Capacitor_SMD:C_0402_1005Metric, symbol Device:C
- added R5: 1-MΩ, Resistor_SMD:R_0402_1005Metric, symbol Device:R
- added U2: LM7805_TO220, Package_TO_SOT_THT:TO-220-3_Vertical, symbol Regulator_Linear:LM7805_TO220
- added U3: LD1117V33, Package_TO_SOT_THT:TO-220-3_Vertical, symbol Regulator_Linear:LD1117V33
- C1: value 1μF -> 100nF; footprint (none) -> Capacitor_SMD:C_0402_1005Metric
- C2, C3, C4: footprint (none) -> Capacitor_SMD:C_0402_1005Metric
- R1, R2, R3, R4: footprint (none) -> Resistor_SMD:R_0402_1005Metric
Connections:
- net IN1N is gone; now on net IN1P: U1.15 (IN1N)
- net AVDD: now also C15.1; no longer U1.19 (AVDD), U1.21 (AVDD), U1.22 (AVDD), U1.56 (AVDD), U1.59 (AVDD)
- net DGND: now also U1.33 (DGND), U1.49 (DGND), U1.51 (DGND); no longer R1.2, R2.2, R3.2, R4.2
- net DVDD: now also C4.2, U1.35 (~{PWDN}), U1.52 (CLKSEL); no longer C4.1, U1.48 (DVDD), U1.50 (DVDD)
- net GND: now also R1.2, R2.2, R3.2, R4.2; no longer C1.2, C2.2, C3.2, C4.2, U1.20 (AVSS), U1.23 (AVSS), U1.32 (AVSS), U1.33 (DGND), U1.49 (DGND), U1.51 (DGND), U1.53 (AVSS1), U1.57 (AVSS), U1.58 (AVSS)
- net at R3.1: now also U1.42 (GPIO1); no longer U1.45 (GPIO3)
- net at R1.1: now also U1.46 (GPIO4); no longer U1.42 (GPIO1)
- net SRB2: now reaches U1.17 (SRB1)
- net SRB1: now reaches U1.18 (SRB2)
- net AVSS: now reaches U1.24 (VREFP)
- net AVSS: now also U1.20 (AVSS), U1.23 (AVSS), U1.32 (AVSS), U1.53 (AVSS1), U1.57 (AVSS), U1.58 (AVSS), C10.1, C11.2, C13.2, C14.1, C7.1, C8.1, C9.1
- net at U1.25 (VREFN): now also C13.1, C14.2
- net at U1.26 (VCAP4): now also C10.2
- net at U1.28 (VCAP1): now also C7.2
- net at U1.30 (VCAP2): now also C8.2
- net AGND: now reaches U1.31 (RESV1)
- net AGND: now also C1.2, C2.2, C3.2, C4.1, U1.41 (DAISY_IN), U1.60 (BIASREF), U1.64 (RESERVED), C15.2, C16.2, C5.1, C6.1, U2.2 (GND), U3.1 (GND)
- net MOSI: now reaches U1.34 (DIN)
- net RESET: now reaches U1.36 (~{RESET})
- net CLK: now reaches U1.37 (CLK)
- net CSI: now reaches U1.39 (~{CS})
- net SCLK: now reaches U1.40 (SCLK)
- net MISO: now reaches U1.43 (DOUT)
- net at R4.1: now also U1.45 (GPIO3); no longer U1.46 (GPIO4)
- net DRDY: now reaches U1.47 (~{DRDY})
- net at U1.55 (VCAP3): now also C11.1, C9.2
- net BIAS_INV: now reaches U1.61 (BIASINV)
- net at U1.62 (BIASIN): now also U1.63 (BIASOUT), C12.1, R5.1
- net AVDD1 renamed Regulator_5V
- net Regulator_5V: now also U1.19 (AVDD), U1.21 (AVDD), U1.22 (AVDD), U1.56 (AVDD), U1.59 (AVDD), C5.2, U2.3 (VO)
- new net +3.7V: U3.3 (VI)
- new net +7.5V: U2.1 (VI)
- new net BIAS_DRV: C12.2, R5.2
- new net Regulator_3.3V: C16.1, C6.2, U1.48 (DVDD), U1.50 (DVDD), U3.2 (VO)
- no-connect marks 0 -> 1
Other:
- note added: "ADS Decoupling"
- note added: "Unipolar"
- note removed: "In Parallel"
- note removed: "USB PWR"
- title: (none) -> EEG ADC BOARD
- moved on the sheet: C4, R4, U1
